File: kicad/pros_rgb/key_group10.kicad_sch (KiCad schematic)
At the start: 16 parts

Commit message: kicad/pros_rgb: minor cleanup
Other:
- note removed: "LD27 0"
- note removed: "LD28 -"
- note removed: "LD44 P"
Changed lines of the file:
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@@
-    (stroke (width 0) (type default) (color 0 0 0 0))
-  )
-  (polyline (pts (xy 144.78 80.01) (xy 149.86 80.01))
     (stroke (width 0) (type default) (color 0 0 0 0))
   )
@@
     (stroke (width 0) (type default) (color 0 0 0 0))
   )
-  (polyline (pts (xy 149.86 49.53) (xy 149.86 54.61))
-    (stroke (width 0) (type default) (color 0 0 0 0))
-  )
   (polyline (pts (xy 251.46 125.73) (xy 251.46 130.81))
     (stroke (width 0) (type default) (color 0 0 0 0))
@@
     (stroke (width 0) (type default) (color 0 0 0 0))
   )
-  (polyline (pts (xy 144.78 80.01) (xy 144.78 74.93))
-    (stroke (width 0) (type default) (color 0 0 0 0))
-  )
   (polyline (pts (xy 106.68 29.21) (xy 106.68 24.13))
     (stroke (width 0) (type default) (color 0 0 0 0))
@@
     (stroke (width 0) (type default) (color 0 0 0 0))
   )
-  (polyline (pts (xy 144.78 54.61) (xy 149.86 54.61))
-    (stroke (width 0) (type default) (color 0 0 0 0))
-  )
   (polyline (pts (xy 271.78 54.61) (xy 276.86 54.61))
     (stroke (width 0) (type default) (color 0 0 0 0))
@@
     (stroke (width 0) (type default) (color 0 0 0 0))
   )
-  (polyline (pts (xy 132.08 54.61) (xy 132.08 49.53))
-    (stroke (width 0) (type default) (color 0 0 0 0))
-  )
-  (polyline (pts (xy 144.78 49.53) (xy 149.86 49.53))
-    (stroke (width 0) (type default) (color 0 0 0 0))
-  )
   (polyline (pts (xy 276.86 74.93) (xy 276.86 80.01))
     (stroke (width 0) (type default) (color 0 0 0 0))
@@
     (stroke (width 0) (type default) (color 0 0 0 0))
   )
-  (polyline (pts (xy 132.08 49.53) (xy 137.16 49.53))
-    (stroke (width 0) (type default) (color 0 0 0 0))
-  )
   (polyline (pts (xy 83.82 151.13) (xy 88.9 151.13))
     (stroke (width 0) (type default) (color 0 0 0 0))
@@
     (stroke (width 0) (type default) (color 0 0 0 0))
   )
-  (polyline (pts (xy 149.86 74.93) (xy 149.86 80.01))
-    (stroke (width 0) (type default) (color 0 0 0 0))
-  )
   (polyline (pts (xy 200.66 74.93) (xy 200.66 80.01))
     (stroke (width 0) (type default) (color 0 0 0 0))
@@
     (stroke (width 0) (type default) (color 0 0 0 0))
   )
-  (polyline (pts (xy 144.78 54.61) (xy 144.78 49.53))
-    (stroke (width 0) (type default) (color 0 0 0 0))
-  )
   (polyline (pts (xy 220.98 100.33) (xy 226.06 100.33))
     (stroke (width 0) (type default) (color 0 0 0 0))
@@
     (stroke (width 0) (type default) (color 0 0 0 0))
   )
-  (polyline (pts (xy 132.08 54.61) (xy 137.16 54.61))
-    (stroke (width 0) (type default) (color 0 0 0 0))
-  )
   (polyline (pts (xy 170.18 74.93) (xy 175.26 74.93))
     (stroke (width 0) (type default) (color 0 0 0 0))
@@
     (stroke (width 0) (type default) (color 0 0 0 0))
   )
-  (polyline (pts (xy 137.16 49.53) (xy 137.16 54.61))
-    (stroke (width 0) (type default) (color 0 0 0 0))
-  )
   (polyline (pts (xy 144.78 29.21) (xy 144.78 24.13))
     (stroke (width 0) (type default) (color 0 0 0 0))
@@
     (stroke (width 0) (type default) (color 0 0 0 0))
   )
-  (polyline (pts (xy 144.78 74.93) (xy 149.86 74.93))
-    (stroke (width 0) (type default) (color 0 0 0 0))
-  )
   (polyline (pts (xy 213.36 74.93) (xy 213.36 80.01))
     (stroke (width 0) (type default) (color 0 0 0 0))
@@
     (effects (font (size 1.27 1.27)) (justify left bottom))
   )
-  (text "LD27\n0" (at 144.78 54.61 0)
-    (effects (font (size 1.27 1.27)) (justify left bottom))
-  )
   (text "LD66\nC" (at 208.28 130.81 0)
     (effects (font (size 1.27 1.27)) (justify left bottom))
@@
     (effects (font (size 1.27 1.27)) (justify left bottom))
   )
-  (text "LD44\nP" (at 144.78 80.01 0)
-    (effects (font (size 1.27 1.27)) (justify left bottom))
-  )
   (text "LD21\n4" (at 220.98 54.61 0)
     (effects (font (size 1.27 1.27)) (justify left bottom))
@@
     (effects (font (size 1.27 1.27)) (justify left bottom))
   )
-  (text "LD28\n-" (at 132.08 54.61 0)
-    (effects (font (size 1.27 1.27)) (justify left bottom))
-  )
