File: kicad/pros_rgb/key_switches.kicad_sch (KiCad schematic)
At the start: 0 parts

Commit message: kicad/pros_rgb: minor cleanup
Other:
- note removed: "LD1 Esc"
- note removed: "LD10 F9"
- note removed: "LD11 F10"
- note removed: "LD12 F11"
- note removed: "LD13 F12"
- note removed: "LD14 PrtSc"
- note removed: "LD15 ScrLk"
- note removed: "LD16 Pause"
- note removed: "LD17 `"
- note removed: "LD18 1"
- note removed: "LD19 2"
- note removed: "LD2 F1"
- note removed: "LD20 3"
- note removed: "LD21 4"
- note removed: "LD22 5"
- note removed: "LD23 6"
- note removed: "LD24 7"
- note removed: "LD25 8"
- note removed: "LD26 9"
- note removed: "LD27 0"
- note removed: "LD28 -"
- note removed: "LD29 ="
- note removed: "LD3 F2"
- note removed: "LD30 Bcksp"
- note removed: "LD31 Ins"
- note removed: "LD32 Home"
- note removed: "LD33 PgUp"
- note removed: "LD34 Tab"
- note removed: "LD35 Q"
- note removed: "LD36 W"
- note removed: "LD37 E"
- note removed: "LD38 R"
- note removed: "LD39 T"
- note removed: "LD4 F3"
- note removed: "LD40 Y"
- note removed: "LD41 U"
- note removed: "LD42 I"
- note removed: "LD43 O"
- note removed: "LD44 P"
- note removed: "LD45 ["
- note removed: "LD46 ]"
- note removed: "LD47 Del"
- note removed: "LD48 End"
- note removed: "LD49 PgDwn"
- note removed: "LD5 F4"
- note removed: "LD50 CapsLk"
- note removed: "LD51 A"
- note removed: "LD52 S"
- note removed: "LD53 D"
- note removed: "LD54 F"
- note removed: "LD55 G"
- note removed: "LD56 H"
- note removed: "LD57 J"
- note removed: "LD58 K"
- note removed: "LD59 L"
- note removed: "LD6 F5"
- note removed: "LD60 ;"
- note removed: "LD61 '"
- note removed: "LD62 Enter"
- note removed: "LD63 LftShift"
- note removed: "LD64 Z"
- note removed: "LD65 X"
- note removed: "LD66 C"
- note removed: "LD67 V"
- note removed: "LD68 B"
- note removed: "LD69 N"
- note removed: "LD7 F6"
- note removed: "LD70 M"
- note removed: "LD71 ,"
- note removed: "LD72 ."
- note removed: "LD73 /"
- note removed: "LD74 RgtShift"
- note removed: "LD75 LftCtrl"
- note removed: "LD76 LftWin"
- note removed: "LD77 LftAlt"
- note removed: "LD78 Space"
- note removed: "LD79 RgtAlt"
- note removed: "LD8 F7"
- note removed: "LD80 RgtWin"
- note removed: "LD81 Fn"
- note removed: "LD82 LftCtrl"
- note removed: "LD83 UpArw"
- note removed: "LD84 DwnArw"
- note removed: "LD85 LftArw"
- note removed: "LD86 RgtArw"
- note removed: "LD87 \"
- note removed: "LD88 NC"
- note removed: "LD89 NC"
- note removed: "LD9 F7"
- note removed: "LD90 NC"
- note removed: "LD91 NC"
- note removed: "LD92 NC"
- note removed: "LD93 NC"
- note removed: "PA5"
- note removed: "PA6"
- note removed: "PA7"
- note removed: "PC11"
- note removed: "PC13"
- note removed: "PC14"
- note removed: "PC15"
- note removed: "PC9"
